File: gassensor_lora_v1/gassensor_lora_v1.kicad_pcb (KiCad board)
At the start: 2 copper layers, 16 parts, among them J1 Conn_01x04, J2 Conn_01x04, SW1 SW_Push, U1 RN2483A, U2 LTC1050

Commit message: add report
Parts:
- removed R1: 10k, Resistor_THT:R_Axial_DIN0204_L3.6mm_D1.6mm_P7.62mm_Horizontal
- removed SW1: SW_Push, Button_Switch_THT:SW_PUSH_6mm
Routing:
- net D2: track 28.1 -> 0.00 mm
- net Net-(R1-Pad1): track 12.3 -> 0.00 mm
- net +5V: track 61.9 -> 62.6 mm
